Commit message: genesis_firefly: B1 — dual-arm URDF imports + reusable Genesis loader
- Made the dual URDF self-contained: rewrote absolute RoboLab mesh paths -> relative to the URDF
  (no cross-repo filesystem dependency). Loads in Genesis: 25 links / 16 joints / 16 dofs.
- robots/firefly_dual.py: Genesis loader. KEY finding (R4): Genesis INTERLEAVES dual-arm dofs
  (left_joint_1=dof0, right_joint_1=dof1, ...) so the layout is NOT contiguous -> we map joint
  NAMES->dof idx (mandatory). Exposes 14-D STATE_JOINTS_14, MIT-controller PD gains/effort limits,
  GR100 open/close/mimic (action-layer coupling), home pose, ee_pose() (with .cpu() at the boundary).
- Verified: home pose renders cleanly, EE links symmetric at [0.16, +/-0.224, 0.276] (base offsets reproduce).

Co-Authored-By: Claude Opus 4.8 (1M context) <noreply@anthropic.com>

File: genesis_firefly/assets/robots/firefly_y6_gr100/dual_firefly_y6_gr100.urdf (robot description, URDF)
Before this commit: robot dual_firefly_y6_gr100, 25 links, 24 joints
Links:
- link left_base_link: geometry collision mesh filename=source/xpkg_urdf_firefly_y6/meshes/base_link.STL; visual mesh filename=source/xpkg_urdf_firefly_y6/meshes/base_link.STL
- link left_camera_body: geometry collision box size=0.023 0.042 0.042; visual mesh filename=source/firefly_y6/d405.stl scale=0.001 0.001 0.001
- link left_gripper_base_link: geometry collision mesh filename=source/xpkg_urdf_gr100/meshes/base_link.STL; visual mesh filename=source/xpkg_urdf_gr100/meshes/base_link.STL
- link left_gripper_left_link_1: geometry collision mesh filename=source/xpkg_urdf_gr100/meshes/L1.STL; visual mesh filename=source/xpkg_urdf_gr100/meshes/L1.STL
- link left_gripper_right_link_1: geometry collision mesh filename=source/xpkg_urdf_gr100/meshes/L2.STL; visual mesh filename=source/xpkg_urdf_gr100/meshes/L2.STL
- link left_link_1: geometry collision mesh filename=source/xpkg_urdf_firefly_y6/meshes/link_1.STL; visual mesh filename=source/xpkg_urdf_firefly_y6/meshes/link_1.STL
- link left_link_2: geometry collision mesh filename=source/xpkg_urdf_firefly_y6/meshes/link_2.STL; visual mesh filename=source/xpkg_urdf_firefly_y6/meshes/link_2.STL
- link left_link_3: geometry collision mesh filename=source/xpkg_urdf_firefly_y6/meshes/link_3.STL; visual mesh filename=source/xpkg_urdf_firefly_y6/meshes/link_3.STL
- link left_link_4: geometry collision mesh filename=source/xpkg_urdf_firefly_y6/meshes/link_4.STL; visual mesh filename=source/xpkg_urdf_firefly_y6/meshes/link_4.STL
- link left_link_5: geometry collision mesh filename=source/xpkg_urdf_firefly_y6/meshes/link_5.STL; visual mesh filename=source/xpkg_urdf_firefly_y6/meshes/link_5.STL
- link left_link_6: geometry collision mesh filename=source/xpkg_urdf_firefly_y6/meshes/link_6.STL; visual mesh filename=source/xpkg_urdf_firefly_y6/meshes/link_6.STL
- link right_base_link: geometry collision mesh filename=source/xpkg_urdf_firefly_y6/meshes/base_link.STL; visual mesh filename=source/xpkg_urdf_firefly_y6/meshes/base_link.STL
- link right_camera_body: geometry collision box size=0.023 0.042 0.042; visual mesh filename=source/firefly_y6/d405.stl scale=0.001 0.001 0.001
- link right_gripper_base_link: geometry collision mesh filename=source/xpkg_urdf_gr100/meshes/base_link.STL; visual mesh filename=source/xpkg_urdf_gr100/meshes/base_link.STL
- link right_gripper_left_link_1: geometry collision mesh filename=source/xpkg_urdf_gr100/meshes/L1.STL; visual mesh filename=source/xpkg_urdf_gr100/meshes/L1.STL
- link right_gripper_right_link_1: geometry collision mesh filename=source/xpkg_urdf_gr100/meshes/L2.STL; visual mesh filename=source/xpkg_urdf_gr100/meshes/L2.STL
- link right_link_1: geometry collision mesh filename=source/xpkg_urdf_firefly_y6/meshes/link_1.STL; visual mesh filename=source/xpkg_urdf_firefly_y6/meshes/link_1.STL
- link right_link_2: geometry collision mesh filename=source/xpkg_urdf_firefly_y6/meshes/link_2.STL; visual mesh filename=source/xpkg_urdf_firefly_y6/meshes/link_2.STL
- link right_link_3: geometry collision mesh filename=source/xpkg_urdf_firefly_y6/meshes/link_3.STL; visual mesh filename=source/xpkg_urdf_firefly_y6/meshes/link_3.STL
- link right_link_4: geometry collision mesh filename=source/xpkg_urdf_firefly_y6/meshes/link_4.STL; visual mesh filename=source/xpkg_urdf_firefly_y6/meshes/link_4.STL
- link right_link_5: geometry collision mesh filename=source/xpkg_urdf_firefly_y6/meshes/link_5.STL; visual mesh filename=source/xpkg_urdf_firefly_y6/meshes/link_5.STL
- link right_link_6: geometry collision mesh filename=source/xpkg_urdf_firefly_y6/meshes/link_6.STL; visual mesh filename=source/xpkg_urdf_firefly_y6/meshes/link_6.STL

Commit message: genesis_firefly: B5 — exact SOMA livery (orange/black + SOMA logo + metallic)
Reproduces RoboLab's recolor_firefly_usd.py exactly in Genesis:
- robots/bake_soma_links.py: bakes the link_2/link_3 panel TEXTURE as portable GLBs using the SAME
  planar-UV + face-split logic (y-faces -> panel_silver.png silver+SOMA-logo; x/z-faces -> panel_carbon.png
  orange+carbon). Verified Genesis renders the GLB texture + alignment is correct (not rotated).
- URDF: link_2/link_3 VISUAL meshes -> the SOMA GLBs (collision stays STL).
- robots/livery.py: solid PBR per link (mat_for): metallic SILVER structure, GREY link_4, near-black
  link_6+base, light camera bodies. apply_livery(robot) before scene.build().
- textures/: panel_carbon.png + panel_silver.png (copied) + baked link_{2,3}_soma.glb.
- .gitignore: stop ignoring asset .png (renders still go to output/temp/).

Result render (genesis_firefly/output/temp/b5_livery) matches firefly_arm_soma_v2.png.

Co-Authored-By: Claude Opus 4.8 (1M context) <noreply@anthropic.com>

File: genesis_firefly/assets/robots/firefly_y6_gr100/dual_firefly_y6_gr100.urdf (robot description, URDF)
Before this commit: robot dual_firefly_y6_gr100, 25 links, 24 joints
Links:
- link left_link_2: geometry collision mesh filename=source/xpkg_urdf_firefly_y6/meshes/link_2.STL; visual mesh filename=textures/link_2_soma.glb
- link left_link_3: geometry collision mesh filename=source/xpkg_urdf_firefly_y6/meshes/link_3.STL; visual mesh filename=textures/link_3_soma.glb
- link right_link_2: geometry collision mesh filename=source/xpkg_urdf_firefly_y6/meshes/link_2.STL; visual mesh filename=textures/link_2_soma.glb
- link right_link_3: geometry collision mesh filename=source/xpkg_urdf_firefly_y6/meshes/link_3.STL; visual mesh filename=textures/link_3_soma.glb
