Commit message: Genesis firefly livery locked: silver Y-faces via side-by-side texture atlas
- link_2/3 panels: ONE GLB / ONE material / ONE <visual> atlas (carbon left, silver strip right) —
  works around Nyx rendering only the first visual + one material per GLB in a URDF subscene.
  Carbon on +/-X,+/-Z (unchanged); +/-Y 'Y faces' = neutral silver (185,186,188).
- Gripper: dark-green fingers, black root, black cap (link_4), dark wrist; arm = brushed silver.
- bake_soma_panels.py / bake_firefly_livery.py = the livery bakers; matte entity-surface override
  kills the warm-env mirror so silver reads neutral in any HDRI.
- Side D435i camera body + support stick (add_side_camera_rig); Nyx photoreal collector (WIP).

Co-Authored-By: Claude Opus 4.8 (1M context) <noreply@anthropic.com>

File: genesis_firefly/assets/robots/firefly_y6_gr100/dual_firefly_y6_gr100_livery.urdf (robot description, URDF)
Before this commit: robot dual_firefly_y6_gr100, 25 links, 24 joints
Links:
- link left_base_link: geometry collision mesh filename=source/xpkg_urdf_firefly_y6/meshes/base_link.STL; visual mesh filename=livery/base_link__dark.glb
- link left_camera_body: geometry collision box size=0.023 0.042 0.042; visual mesh filename=livery/d405__camg.glb scale=0.001 0.001 0.001
- link left_gripper_base_link: geometry collision mesh filename=source/xpkg_urdf_gr100/meshes/base_link.STL; visual mesh filename=livery/base_link__black.glb
- link left_gripper_left_link_1: geometry collision mesh filename=source/xpkg_urdf_gr100/meshes/L1_pad.STL; visual mesh filename=livery/L1__green.glb
- link left_gripper_right_link_1: geometry collision mesh filename=source/xpkg_urdf_gr100/meshes/L2_pad.STL; visual mesh filename=livery/L2__green.glb
- link left_link_1: geometry collision mesh filename=source/xpkg_urdf_firefly_y6/meshes/link_1.STL; visual mesh filename=livery/link_1__silver.glb
- link left_link_4: geometry collision mesh filename=source/xpkg_urdf_firefly_y6/meshes/link_4.STL; visual mesh filename=livery/link_4__black.glb
- link left_link_5: geometry collision mesh filename=source/xpkg_urdf_firefly_y6/meshes/link_5.STL; visual mesh filename=livery/link_5__silver.glb
- link left_link_6: geometry collision mesh filename=source/xpkg_urdf_firefly_y6/meshes/link_6.STL; visual mesh filename=livery/link_6__dark.glb
- link right_base_link: geometry collision mesh filename=source/xpkg_urdf_firefly_y6/meshes/base_link.STL; visual mesh filename=livery/base_link__dark.glb
- link right_camera_body: geometry collision box size=0.023 0.042 0.042; visual mesh filename=livery/d405__camg.glb scale=0.001 0.001 0.001
- link right_gripper_base_link: geometry collision mesh filename=source/xpkg_urdf_gr100/meshes/base_link.STL; visual mesh filename=livery/base_link__black.glb
- link right_gripper_left_link_1: geometry collision mesh filename=source/xpkg_urdf_gr100/meshes/L1_pad.STL; visual mesh filename=livery/L1__green.glb
- link right_gripper_right_link_1: geometry collision mesh filename=source/xpkg_urdf_gr100/meshes/L2_pad.STL; visual mesh filename=livery/L2__green.glb
- link right_link_1: geometry collision mesh filename=source/xpkg_urdf_firefly_y6/meshes/link_1.STL; visual mesh filename=livery/link_1__silver.glb
- link right_link_4: geometry collision mesh filename=source/xpkg_urdf_firefly_y6/meshes/link_4.STL; visual mesh filename=livery/link_4__black.glb
- link right_link_5: geometry collision mesh filename=source/xpkg_urdf_firefly_y6/meshes/link_5.STL; visual mesh filename=livery/link_5__silver.glb
- link right_link_6: geometry collision mesh filename=source/xpkg_urdf_firefly_y6/meshes/link_6.STL; visual mesh filename=livery/link_6__dark.glb
